Commit message: Alignment with the paper
Signed-off-by: root <root@LAPTOP-55B7T539>

File: ur_description/urdf/ur5.urdf (robot description, URDF)
Before this commit: robot ur5_robot, 11 links, 10 joints
Joints:
- joint base_link-base_fixed_joint: origin xyz=0 0 0 rpy=0 0 3.141592653589793 -> xyz=0 0 0 rpy=0 0 0

Commit message: EE->Task into the model & bug fixing
Signed-off-by: root <root@LAPTOP-55B7T539>

File: ur_description/urdf/ur5.urdf (robot description, URDF)
Before this commit: robot ur5_robot, 11 links, 10 joints
Joints:
- joint base_link-base_link_inertia: origin xyz=0 0 0 rpy=0 0 3.141592653589793 -> xyz=0 0 0 rpy=0 0 0
- joint shoulder_pan_joint: origin xyz=0 0 0.089159 rpy=0 0 0 -> xyz=0 0 0.089159 rpy=0 0 3.141592653589793

Commit message: Plotting for report

File: ur_description/urdf/ur5.urdf (robot description, URDF)
Before this commit: robot ur5_robot, 11 links, 10 joints
Links:
- link base_link_inertia: geometry collision mesh filename=package://ur_description/meshes/collision/base.stl; visual mesh filename=package://ur_description/meshes/visual/base.dae
- link forearm_link: geometry collision mesh filename=package://ur_description/meshes/collision/forearm.stl; visual mesh filename=package://ur_description/meshes/visual/forearm.dae
- link shoulder_link: geometry collision mesh filename=package://ur_description/meshes/collision/shoulder.stl; visual mesh filename=package://ur_description/meshes/visual/shoulder.dae
- link upper_arm_link: geometry collision mesh filename=package://ur_description/meshes/collision/upperarm.stl; visual mesh filename=package://ur_description/meshes/visual/upperarm.dae
- link wrist_1_link: geometry collision mesh filename=package://ur_description/meshes/collision/wrist1.stl; visual mesh filename=package://ur_description/meshes/visual/wrist1.dae
- link wrist_2_link: geometry collision mesh filename=package://ur_description/meshes/collision/wrist2.stl; visual mesh filename=package://ur_description/meshes/visual/wrist2.dae
- link wrist_3_link: geometry collision mesh filename=package://ur_description/meshes/collision/wrist3.stl; visual mesh filename=package://ur_description/meshes/visual/wrist3.dae

Commit message: Pushing latest changes before merge with main

File: ur_description/urdf/ur5.urdf (robot description, URDF)
Before this commit: robot ur5_robot, 11 links, 10 joints
Links:
- link base_link_inertia: geometry collision mesh filename=package://ur_description/meshes/ur5/collision/base.stl; visual mesh filename=package://ur_description/meshes/ur5/visual/Base.dae
- link forearm_link: geometry collision mesh filename=package://ur_description/meshes/ur5/collision/forearm.stl; visual mesh filename=package://ur_description/meshes/ur5/visual/Forearm.dae
- link shoulder_link: geometry collision mesh filename=package://ur_description/meshes/ur5/collision/shoulder.stl; visual mesh filename=package://ur_description/meshes/ur5/visual/Shoulder.dae
- link upper_arm_link: geometry collision mesh filename=package://ur_description/meshes/ur5/collision/upper_arm.stl; visual mesh filename=package://ur_description/meshes/ur5/visual/UpperArm.dae
- link wrist_1_link: geometry collision mesh filename=package://ur_description/meshes/ur5/collision/wrist_1.stl; visual mesh filename=package://ur_description/meshes/ur5/visual/Wrist1.dae
- link wrist_2_link: geometry collision mesh filename=package://ur_description/meshes/ur5/collision/wrist_2.stl; visual mesh filename=package://ur_description/meshes/ur5/visual/Wrist2.dae
- link wrist_3_link: geometry collision mesh filename=package://ur_description/meshes/ur5/collision/wrist_3.stl; visual mesh filename=package://ur_description/meshes/ur5/visual/Wrist3.dae
